File: pcb/Sensing Device/Sensing Device.kicad_sch (KiCad schematic)
At the start: 19 parts, among them J1 PWR_PAD, J2 ID_PAD, SW1 SW_SPST, SW2 SW_SPDT, U2 TLV493D

Commit message: datasheet
Parts:
- BT1: value Lipo battery -> 3.7v Lipo battery
- R1, R3: value 4.7kΩ -> 4.3kΩ
Connections:
- net 3V3: now also C2.1, C3.1, R1.2, R4.2, R6.2, U2.4 (VDD)
- net VCC: no longer C2.1, C3.1, R1.2, R4.2, R6.2, U2.4 (VDD)
Other:
- company: (none) -> Leo Peng
- title: (none) -> MagDocker Tangible Input Device
Changed lines of the file:
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@@
 (kicad_sch (version 20230121) (generator eeschema)
   (paper "A4")
+  (title_block
+    (title "MagDocker Tangible Input Device")
+    (date "2024-01-27")
+    (rev "V1.0")
+    (company "Leo Peng")
+    (comment 1 "processes the data on ESP32S3 and sends it to computer via BLE communication")
+    (comment 2 "which reads 3-axis magnetic field information via TLV493D,")
+    (comment 3 "This is the PCB of the sensing device of MagDocker, ")
+    (comment 4 " ")
+  )
   (junction (at 123.19 140.97) (diameter 0) (color 0 0 0 0)
   )
@@
     (stroke (width 0) (type default))
   )
+  (wire (pts (xy 48.26 130.81) (xy 48.26 132.08))
+    (stroke (width 0) (type default))
+  )
   (wire (pts (xy 123.19 151.13) (xy 123.19 153.67))
     (stroke (width 0) (type default))
@@
     (effects (font (size 1.27 1.27)) (justify left bottom))
   )
+  (label "3V3" (at 48.26 130.81 0) (fields_autoplaced)
+    (effects (font (size 1.27 1.27)) (justify left bottom))
+  )
   (label "Id" (at 127 140.97 0) (fields_autoplaced)
     (effects (font (size 1.27 1.27)) (justify left bottom))
@@
     (effects (font (size 1.27 1.27)) (justify right bottom))
   )
+  (label "3V3" (at 269.24 66.04 0) (fields_autoplaced)
+    (effects (font (size 1.27 1.27)) (justify left bottom))
+  )
   (label "SCL_XIAO" (at 95.25 90.17 180) (fields_autoplaced)
     (effects (font (size 1.27 1.27)) (justify right bottom))
@@
     (effects (font (size 1.27 1.27)) (justify right bottom))
   )
+  (label "3V3" (at 255.27 66.04 0) (fields_autoplaced)
+    (effects (font (size 1.27 1.27)) (justify left bottom))
+  )
   (label "SDA_TLV" (at 172.72 96.52 180) (fields_autoplaced)
     (effects (font (size 1.27 1.27)) (justify right bottom))
@@
     (effects (font (size 1.27 1.27)) (justify left bottom))
   )
+  (label "3V3" (at 234.95 66.04 0) (fields_autoplaced)
+    (effects (font (size 1.27 1.27)) (justify left bottom))
+  )
   (label "SCL_TLV" (at 217.17 77.47 0) (fields_autoplaced)
+    (effects (font (size 1.27 1.27)) (justify left bottom))
+  )
+  (label "3V3" (at 172.72 66.04 0) (fields_autoplaced)
     (effects (font (size 1.27 1.27)) (justify left bottom))
   )
@@
     (effects (font (size 1.27 1.27)) (justify right bottom))
   )
+  (label "3V3" (at 200.66 66.04 0) (fields_autoplaced)
+    (effects (font (size 1.27 1.27)) (justify left bottom))
+  )
   (label "3V3" (at 147.32 82.55 0) (fields_autoplaced)
     (effects (font (size 1.27 1.27)) (justify left bottom))
@@
         (path "/51ce3d25-026d-4dec-aec0-5bd74cd3b771"
           (reference "D1") (unit 1)
-        )
-      )
-    )
-  )
-  (symbol (lib_id "power:VCC") (at 269.24 66.04 0) (unit 1)
-    (in_bom yes) (on_board yes) (dnp no) (fields_autoplaced)
-    (property "Reference" "#PWR019" (at 269.24 69.85 0)
-      (effects (font (size 1.27 1.27)) hide)
-    )
-    (property "Value" "VCC" (at 269.24 60.96 0)
-      (effects (font (size 1.27 1.27)))
-    )
-    (property "Footprint" "" (at 269.24 66.04 0)
-      (effects (font (size 1.27 1.27)) hide)
-    )
-    (property "Datasheet" "" (at 269.24 66.04 0)
-      (effects (font (size 1.27 1.27)) hide)
-    )
-    (pin "1")
-    (instances
-      (project "Sensing Device"
-        (path "/51ce3d25-026d-4dec-aec0-5bd74cd3b771"
-          (reference "#PWR019") (unit 1)
-        )
-      )
-    )
-  )
-  (symbol (lib_id "power:VCC") (at 234.95 66.04 0) (unit 1)
-    (in_bom yes) (on_board yes) (dnp no) (fields_autoplaced)
-    (property "Reference" "#PWR015" (at 234.95 69.85 0)
-      (effects (font (size 1.27 1.27)) hide)
-    )
-    (property "Value" "VCC" (at 234.95 60.96 0)
-      (effects (font (size 1.27 1.27)))
-    )
-    (property "Footprint" "" (at 234.95 66.04 0)
-      (effects (font (size 1.27 1.27)) hide)
-    )
-    (property "Datasheet" "" (at 234.95 66.04 0)
-      (effects (font (size 1.27 1.27)) hide)
-    )
-    (pin "1")
-    (instances
-      (project "Sensing Device"
-        (path "/51ce3d25-026d-4dec-aec0-5bd74cd3b771"
-          (reference "#PWR015") (unit 1)
-        )
-      )
-    )
-  )
-  (symbol (lib_id "power:VCC") (at 172.72 66.04 0) (unit 1)
-    (in_bom yes) (on_board yes) (dnp no) (fields_autoplaced)
-    (property "Reference" "#PWR012" (at 172.72 69.85 0)
-      (effects (font (size 1.27 1.27)) hide)
-    )
-    (property "Value" "VCC" (at 172.72 60.96 0)
-      (effects (font (size 1.27 1.27)))
-    )
-    (property "Footprint" "" (at 172.72 66.04 0)
-      (effects (font (size 1.27 1.27)) hide)
-    )
-    (property "Datasheet" "" (at 172.72 66.04 0)
-      (effects (font (size 1.27 1.27)) hide)
-    )
-    (pin "1")
-    (instances
-      (project "Sensing Device"
-        (path "/51ce3d25-026d-4dec-aec0-5bd74cd3b771"
-          (reference "#PWR012") (unit 1)
         )
       )
@@
     )
   )
-  (symbol (lib_id "power:VCC") (at 255.27 66.04 0) (unit 1)
-    (in_bom yes) (on_board yes) (dnp no) (fields_autoplaced)
-    (property "Reference" "#PWR017" (at 255.27 69.85 0)
-      (effects (font (size 1.27 1.27)) hide)
-    )
-    (property "Value" "VCC" (at 255.27 60.96 0)
-      (effects (font (size 1.27 1.27)))
-    )
-    (property "Footprint" "" (at 255.27 66.04 0)
-      (effects (font (size 1.27 1.27)) hide)
-    )
-    (property "Datasheet" "" (at 255.27 66.04 0)
-      (effects (font (size 1.27 1.27)) hide)
-    )
-    (pin "1")
-    (instances
-      (project "Sensing Device"
-        (path "/51ce3d25-026d-4dec-aec0-5bd74cd3b771"
-          (reference "#PWR017") (unit 1)
-        )
-      )
-    )
-  )
   (symbol (lib_id "power:GND") (at 80.01 96.52 0) (unit 1)
     (in_bom yes) (on_board yes) (dnp no) (fields_autoplaced)
@@
     )
   )
-  (symbol (lib_id "power:VCC") (at 48.26 132.08 0) (unit 1)
-    (in_bom yes) (on_board yes) (dnp no) (fields_autoplaced)
-    (property "Reference" "#PWR04" (at 48.26 135.89 0)
-      (effects (font (size 1.27 1.27)) hide)
-    )
-    (property "Value" "VCC" (at 48.26 127 0)
-      (effects (font (size 1.27 1.27)))
-    )
-    (property "Footprint" "" (at 48.26 132.08 0)
-      (effects (font (size 1.27 1.27)) hide)
-    )
-    (property "Datasheet" "" (at 48.26 132.08 0)
-      (effects (font (size 1.27 1.27)) hide)
-    )
-    (pin "1")
-    (instances
-      (project "Sensing Device"
-        (path "/51ce3d25-026d-4dec-aec0-5bd74cd3b771"
-          (reference "#PWR04") (unit 1)
-        )
-      )
-    )
-  )
   (symbol (lib_id "power:GND") (at 255.27 91.44 0) (unit 1)
     (in_bom yes) (on_board yes) (dnp no) (fields_autoplaced)
@@
     )
   )
-  (symbol (lib_id "power:VCC") (at 200.66 66.04 0) (unit 1)
-    (in_bom yes) (on_board yes) (dnp no) (fields_autoplaced)
-    (property "Reference" "#PWR014" (at 200.66 69.85 0)
-      (effects (font (size 1.27 1.27)) hide)
-    )
-    (property "Value" "VCC" (at 200.66 60.96 0)
-      (effects (font (size 1.27 1.27)))
-    )
-    (property "Footprint" "" (at 200.66 66.04 0)
-      (effects (font (size 1.27 1.27)) hide)
-    )
-    (property "Datasheet" "" (at 200.66 66.04 0)
-      (effects (font (size 1.27 1.27)) hide)
-    )
-    (pin "1")
-    (instances
-      (project "Sensing Device"
-        (path "/51ce3d25-026d-4dec-aec0-5bd74cd3b771"
-          (reference "#PWR014") (unit 1)
-        )
-      )
-    )
-  )
   (symbol (lib_id "power:GND") (at 234.95 92.71 0) (unit 1)
     (in_bom yes) (on_board yes) (dnp no) (fields_autoplaced)
@@
   )
   (symbol (lib_id "Device:Battery_Cell") (at 33.02 88.9 0) (unit 1)
-    (in_bom yes) (on_board yes) (dnp no) (fields_autoplaced)
-    (property "Reference" "BT1" (at 36.83 85.7885 0)
-      (effects (font (size 1.27 1.27)) (justify left))
-    )
-    (property "Value" "Lipo battery" (at 36.83 88.3285 0)
+    (in_bom yes) (on_board yes) (dnp no)
+    (property "Reference" "BT1" (at 36.83 87.63 0)
+      (effects (font (size 1.27 1.27)) (justify left))
+    )
+    (property "Value" "3.7v Lipo battery" (at 34.29 90.17 0)
       (effects (font (size 1.27 1.27)) (justify left))
     )
@@
       (effects (font (size 1.27 1.27)) (justify right))
     )
-    (property "Value" "4.7kΩ" (at 50.8 137.16 0)
+    (property "Value" "4.3kΩ" (at 50.8 137.16 0)
       (effects (font (size 1.27 1.27)) (justify right))
     )
@@
       (effects (font (size 1.27 1.27)) (justify right))
     )
-    (property "Value" "4.7kΩ" (at 125.73 135.89 0)
+    (property "Value" "4.3kΩ" (at 125.73 135.89 0)
       (effects (font (size 1.27 1.27)) (justify right))
     )

Commit message: power management
Parts:
- added C4: 200 pF, Capacitor_SMD:C_0805_2012Metric_Pad1.18x1.45mm_HandSolder, symbol Device:C
- C1: value 100 nF -> 200 pF
- R2: value 470Ω -> 50Ω
Connections:
- net GND: now also C4.2
- net VCC: now also C4.1; no longer D1.2 (A)
- net LED: now reaches U1.4 (GPIO4_A3_D3)
- net LED: now also D1.2 (A)
- no-connect marks 9 -> 8
Other:
- note added: "Notes: Leave C2 and C3 blank and test first. These two capacitors might not be necessary."
- note added: "Notes: Leave C4 blank and test first."
- moved on the sheet: BT1, C1, C2, C3, D1, J1, R2, R4, R5, R6, R7, R8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

Commit message: readme
Parts:
- D1: value LED -> LS R976; footprint LED_THT:LED_D4.0mm -> LED_SMD:LED_0805_2012Metric_Pad1.15x1.40mm_HandSolder
- R2: value 50Ω -> 65Ω
Changed lines of the file:
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@@
       (effects (font (size 1.27 1.27)) (justify right))
     )
-    (property "Value" "LED" (at 55.88 79.0575 90)
+    (property "Value" "LS R976" (at 55.88 79.0575 90)
       (effects (font (size 1.27 1.27)) (justify right))
     )
-    (property "Footprint" "LED_THT:LED_D4.0mm" (at 52.07 76.2 0)
+    (property "Footprint" "LED_SMD:LED_0805_2012Metric_Pad1.15x1.40mm_HandSolder" (at 52.07 76.2 0)
       (effects (font (size 1.27 1.27)) hide)
     )
@@
       (effects (font (size 1.27 1.27)) (justify left))
     )
-    (property "Value" "50Ω" (at 54.61 88.9 0)
-      (effects (font (size 1.27 1.27)) (justify left))
-    )
+    (property "Value" "65Ω" (at 54.61 88.9 0)
+      (effects (font (size 1.27 1.27)) (justify left))
+    )
