File: pcb/Sensing Device/Sensing Device.kicad_pcb (KiCad board)
At the start: 2 copper layers, 100 x 60 mm, 19 parts, among them J1 PWR_PAD, J2 ID_PAD, SW1 SW_SPST, SW2 SW_SPDT, U2 TLV493D

Commit message: datasheet
Parts:
- BT1: value Lipo battery -> 3.7v Lipo battery
- R1, R3: value 4.7kΩ -> 4.3kΩ
Connections:
- C2 pad 1: VCC -> /3V3
- C3 pad 1: VCC -> /3V3
- R1 pad 2: VCC -> /3V3
- R4 pad 2: VCC -> /3V3
- R6 pad 2: VCC -> /3V3
- U2 pad 4: VCC -> /3V3
Routing:
- net /3V3: track 51.3 -> 253.2 mm, vias 0 -> 1
- net VCC: track 260.5 -> 66.4 mm, vias 1 -> 0
- net GND: track 197.4 -> 204.2 mm
Other:
- board text added: "Leo Peng MagDocker v1.0"

Commit message: power management
Parts:
- added C4: 200 pF, Capacitor_SMD:C_0805_2012Metric_Pad1.18x1.45mm_HandSolder, F.Cu at (84.1, 64.8)
- C1: value 100 nF -> 200 pF
- R2: value 470Ω -> 50Ω
- turned C2 to 90 degrees
- turned C3 to 90 degrees
Connections:
- D1 pad 2: VCC -> /LED
- U1 pad 4: unconnected-(U1-GPIO4_A3_D3-Pad4) -> /LED
Routing:
- net VCC: track 66.4 -> 40.2 mm
- net /LED: track 0.00 -> 16.7 mm
- net GND: track 204.2 -> 210.6 mm
- net /3V3: track 253.2 -> 251.3 mm
- net /Button: track 59.5 -> 60.6 mm
Other:
- board text added: "PP MagDocker v2.0"
- board text removed: "Leo Peng MagDocker v1.0"

Commit message: readme
Parts:
- D1: value LED -> LS R976; footprint LED_THT:LED_D4.0mm -> LED_SMD:LED_0805_2012Metric_Pad1.15x1.40mm_HandSolder
- R2: value 50Ω -> 65Ω
- moved BT1 10.9 mm to (84.1, 81.8), turned to 0 degrees
- moved SW1 1.39 mm to (64.8, 67.5)
- moved SW2 0.76 mm to (91.8, 98.0)
Routing:
- net VCC: track 40.2 -> 54.3 mm
- net Net-(BT1-+): track 16.5 -> 23.3 mm, vias 0 -> 1
- net GND: track 210.6 -> 205.0 mm, vias 0 -> 1
- net Net-(C1-Pad1): track 53.8 -> 52.0 mm
- net /LED: track 16.7 -> 15.2 mm
- net Net-(D1-K): track 4.32 -> 3.29 mm
- net /Button: track 60.6 -> 61.3 mm
Other:
- board size 100 x 60 mm -> 110 x 70 mm
- board text added: "+"
- board text added: "-"
- board text added: "MagDocker @Yuecheng"
- board text removed: "PP MagDocker v2.0"
