File: pcb/Display Device/display_rasp/display_rasp.kicad_sch (KiCad schematic)
At the start: 7 parts, among them J1 Conn_01x04, J2 Conn_01x04, M1 Stepper_Motor_bipolar, SW1 SW_SPST

Commit message: readme
Other:
- title: (none) -> Display Device
Changed lines of the file:
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@@
 (kicad_sch (version 20230121) (generator eeschema)
   (paper "A4")
+  (title_block
+    (title "Display Device")
+    (date "2024-03-05")
+    (rev "Yuecheng Peng")
+  )
   (junction (at 171.45 106.68) (diameter 0) (color 0 0 0 0)
   )
